File: emg-bridge.sch (EAGLE design)
At the start: 24 parts, among them J1 RJ25_4X1, J2 RJ25_4X1, J3 M03_0.156IN-RA, U1 ADM660ARZ

Commit message: Realization: the MC USB-1608G DAQ can only output 10mA for power, so the power circuitry has been completely reworked. Now with 3kV isolation!
Parts:
- removed U1: ADM660ARZ, eagle-lib:ADM660ARZ
- added C3: 0.1uF, SparkFun-Capacitors:CAP0805
- added JP2: USB-B, SparkFun-Connectors:USBPTH
- added U2: DC_ISOLATOR-RKZ0505D, eagle-lib:DC_ISOLATOR-RKZ0505D
- C1, C2: value 10uF -> 0.1uF
Connections:
- net +VE: now also C2.1, U2.+VOUT; no longer JP1.1, U1.V+
- net -VE: now also C3.2, U2.-VOUT; no longer C2.1, U1.OUT
- net GND: now also C3.1, JP1.1, U2.COM; no longer U1.GND, U1.LV
- net N$2: now also C1.1, JP2.VBUS, U2.+VIN; no longer C1.2, U1.CAP-
- net N$4: now also C1.2, JP2.GND, U2.-VIN; no longer C1.1, U1.CAP+
Other:
- moved on the sheet: C1, C2
Changed lines of the file:
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@@
 </classes>
 <parts>
-<part name="C1" library="SparkFun-Capacitors" deviceset="CAP" device="0805" value="10uF"/>
-<part name="C2" library="SparkFun-Capacitors" deviceset="CAP" device="0805" value="10uF"/>
 <part name="R1" library="SparkFun-Passives" deviceset="RESISTOR" device="0805-RES" value="100"/>
 <part name="R2" library="SparkFun-Passives" deviceset="RESISTOR" device="0805-RES" value="100"/>
@@
 <part name="J1" library="eagle-lib" deviceset="RJ25_4X1" device=""/>
 <part name="J2" library="eagle-lib" deviceset="RJ25_4X1" device=""/>
-<part name="GND1" library="SparkFun-Aesthetics" deviceset="GND" device=""/>
-<part name="GND2" library="SparkFun-Aesthetics" deviceset="GND" device=""/>
-<part name="GND3" library="SparkFun-Aesthetics" deviceset="GND" device=""/>
 <part name="GND4" library="SparkFun-Aesthetics" deviceset="GND" device=""/>
 <part name="GND5" library="SparkFun-Aesthetics" deviceset="GND" device=""/>
@@
 <part name="GND12" library="SparkFun-Aesthetics" deviceset="GND" device=""/>
 <part name="GND13" library="SparkFun-Aesthetics" deviceset="GND" device=""/>
-<part name="U1" library="eagle-lib" deviceset="ADM660" device="ARZ"/>
 <part name="J3" library="eagle-lib" deviceset="M03" device="_0.156IN-RA"/>
 <part name="JP1" library="SparkFun-Connectors" deviceset="M05X2" device="RAF"/>
 <part name="FRAME1" library="frames" deviceset="FRAME_A_L" device="" value="FRAME"/>
 <part name="U$1" library="ucdrascal-eagle-lib" deviceset="UCDAVIS-RASCAL_LOGO" device="-2LINE"/>
+<part name="U2" library="eagle-lib" deviceset="DC_ISOLATOR" device="-RKZ0505D"/>
+<part name="JP2" library="SparkFun-Connectors" deviceset="USB" device="PTH" value="USB-B"/>
+<part name="C1" library="SparkFun-Capacitors" deviceset="CAP" device="0805" value="0.1uF"/>
+<part name="C2" library="SparkFun-Capacitors" deviceset="CAP" device="0805" value="0.1uF"/>
+<part name="C3" library="SparkFun-Capacitors" deviceset="CAP" device="0805" value="0.1uF"/>
 </parts>
 <sheets>
@@
 </plain>
 <instances>
-<instance part="C1" gate="G$1" x="162.56" y="149.86"/>
-<instance part="C2" gate="G$1" x="220.98" y="144.78"/>
 <instance part="R1" gate="G$1" x="55.88" y="160.02"/>
 <instance part="R2" gate="G$1" x="55.88" y="152.4"/>
@@
 <instance part="J2" gate="C" x="83.82" y="109.22"/>
 <instance part="J2" gate="D" x="83.82" y="83.82"/>
-<instance part="GND1" gate="1" x="213.36" y="137.16"/>
-<instance part="GND2" gate="1" x="175.26" y="137.16"/>
-<instance part="GND3" gate="1" x="220.98" y="137.16"/>
 <instance part="GND4" gate="1" x="43.18" y="147.32"/>
 <instance part="GND5" gate="1" x="43.18" y="121.92"/>
@@
 <instance part="GND12" gate="1" x="170.18" y="78.74"/>
 <instance part="GND13" gate="1" x="243.84" y="78.74"/>
-<instance part="U1" gate="G$1" x="195.58" y="157.48"/>
 <instance part="J3" gate="G$1" x="157.48" y="91.44"/>
 <instance part="JP1" gate="G$1" x="226.06" y="88.9"/>
@@
 <instance part="FRAME1" gate="G$2" x="172.72" y="0"/>
 <instance part="U$1" gate="G$1" x="180.34" y="40.64"/>
+<instance part="U2" gate="G$1" x="200.66" y="147.32"/>
+<instance part="JP2" gate="G$1" x="167.64" y="149.86" rot="MR0"/>
+<instance part="C1" gate="G$1" x="180.34" y="147.32"/>
+<instance part="C2" gate="G$1" x="218.44" y="149.86"/>
+<instance part="C3" gate="G$1" x="220.98" y="142.24"/>
 </instances>
 <busses>
@@
 <wire x1="243.84" y1="81.28" x2="243.84" y2="93.98" width="0.1524" layer="91"/>
 <pinref part="JP1" gate="G$1" pin="2"/>
+<pinref part="JP1" gate="G$1" pin="1"/>
+<wire x1="218.44" y1="93.98" x2="215.9" y2="93.98" width="0.1524" layer="91"/>
+<wire x1="215.9" y1="93.98" x2="215.9" y2="101.6" width="0.1524" layer="91"/>
+<wire x1="215.9" y1="101.6" x2="243.84" y2="101.6" width="0.1524" layer="91"/>
+<wire x1="243.84" y1="101.6" x2="243.84" y2="93.98" width="0.1524" layer="91"/>
+<junction x="243.84" y="93.98"/>
 </segment>
 <segment>
@@
 </segment>
 <segment>
-<pinref part="GND2" gate="1" pin="GND"/>
-<wire x1="175.26" y1="139.7" x2="175.26" y2="154.94" width="0.1524" layer="91"/>
-<wire x1="175.26" y1="154.94" x2="180.34" y2="154.94" width="0.1524" layer="91"/>
-<pinref part="U1" gate="G$1" pin="GND"/>
-</segment>
-<segment>
-<pinref part="GND1" gate="1" pin="GND"/>
-<wire x1="210.82" y1="154.94" x2="213.36" y2="154.94" width="0.1524" layer="91"/>
-<wire x1="213.36" y1="154.94" x2="213.36" y2="139.7" width="0.1524" layer="91"/>
-<pinref part="U1" gate="G$1" pin="LV"/>
-</segment>
-<segment>
-<pinref part="GND3" gate="1" pin="GND"/>
-<pinref part="C2" gate="G$1" pin="2"/>
-<wire x1="220.98" y1="139.7" x2="220.98" y2="142.24" width="0.1524" layer="91"/>
-</segment>
-<segment>
 <pinref part="GND6" gate="1" pin="GND"/>
 <wire x1="43.18" y1="99.06" x2="43.18" y2="106.68" width="0.1524" layer="91"/>
@@
 <wire x1="43.18" y1="106.68" x2="43.18" y2="114.3" width="0.1524" layer="91"/>
 </segment>
+<segment>
+<pinref part="U2" gate="G$1" pin="COM"/>
+<wire x1="215.9" y1="147.32" x2="218.44" y2="147.32" width="0.1524" layer="91"/>
+<label x="231.14" y="147.32" size="1.778" layer="95"/>
+<pinref part="C2" gate="G$1" pin="2"/>
+<wire x1="218.44" y1="147.32" x2="220.98" y2="147.32" width="0.1524" layer="91"/>
+<junction x="218.44" y="147.32"/>
+<pinref part="C3" gate="G$1" pin="1"/>
+<wire x1="220.98" y1="147.32" x2="233.68" y2="147.32" width="0.1524" layer="91"/>
+<junction x="220.98" y="147.32"/>
+</segment>
 </net>
 <net name="CH1" class="0">
@@
 </segment>
 <segment>
-<wire x1="210.82" y1="160.02" x2="231.14" y2="160.02" width="0.1524" layer="91"/>
-<label x="226.06" y="160.02" size="1.778" layer="95"/>
-<pinref part="U1" gate="G$1" pin="V+"/>
-</segment>
-<segment>
-<wire x1="218.44" y1="93.98" x2="208.28" y2="93.98" width="0.1524" layer="91"/>
-<label x="208.28" y="99.06" size="1.778" layer="95"/>
-<wire x1="208.28" y1="93.98" x2="208.28" y2="99.06" width="0.1524" layer="91"/>
-<pinref part="JP1" gate="G$1" pin="1"/>
+<pinref part="U2" gate="G$1" pin="+VOUT"/>
+<wire x1="215.9" y1="154.94" x2="218.44" y2="154.94" width="0.1524" layer="91"/>
+<label x="231.14" y="154.94" size="1.778" layer="95"/>
+<pinref part="C2" gate="G$1" pin="1"/>
+<wire x1="218.44" y1="154.94" x2="233.68" y2="154.94" width="0.1524" layer="91"/>
+<junction x="218.44" y="154.94"/>
 </segment>
 </net>
@@
 </segment>
 <segment>
-<wire x1="210.82" y1="152.4" x2="220.98" y2="152.4" width="0.1524" layer="91"/>
-<pinref part="C2" gate="G$1" pin="1"/>
-<wire x1="220.98" y1="149.86" x2="220.98" y2="152.4" width="0.1524" layer="91"/>
-<wire x1="220.98" y1="152.4" x2="231.14" y2="152.4" width="0.1524" layer="91"/>
-<junction x="220.98" y="152.4"/>
-<label x="226.06" y="152.4" size="1.778" layer="95"/>
-<pinref part="U1" gate="G$1" pin="OUT"/>
+<pinref part="U2" gate="G$1" pin="-VOUT"/>
+<wire x1="215.9" y1="139.7" x2="220.98" y2="139.7" width="0.1524" layer="91"/>
+<label x="231.14" y="139.7" size="1.778" layer="95"/>
+<pinref part="C3" gate="G$1" pin="2"/>
+<wire x1="220.98" y1="139.7" x2="233.68" y2="139.7" width="0.1524" layer="91"/>
+<junction x="220.98" y="139.7"/>
 </segment>
 </net>
 <net name="N$2" class="0">
 <segment>
-<wire x1="180.34" y1="152.4" x2="172.72" y2="152.4" width="0.1524" layer="91"/>
-<wire x1="172.72" y1="152.4" x2="172.72" y2="144.78" width="0.1524" layer="91"/>
-<wire x1="172.72" y1="144.78" x2="162.56" y2="144.78" width="0.1524" layer="91"/>
-<wire x1="162.56" y1="144.78" x2="162.56" y2="147.32" width="0.1524" layer="91"/>
+<pinref part="JP2" gate="G$1" pin="VBUS"/>
+<pinref part="C1" gate="G$1" pin="1"/>
+<wire x1="170.18" y1="152.4" x2="180.34" y2="152.4" width="0.1524" layer="91"/>
+<pinref part="U2" gate="G$1" pin="+VIN"/>
+<wire x1="180.34" y1="152.4" x2="185.42" y2="152.4" width="0.1524" layer="91"/>
+<junction x="180.34" y="152.4"/>
+</segment>
+</net>
+<net name="N$4" class="0">
+<segment>
+<pinref part="JP2" gate="G$1" pin="GND"/>
+<wire x1="170.18" y1="149.86" x2="175.26" y2="149.86" width="0.1524" layer="91"/>
+<wire x1="175.26" y1="149.86" x2="175.26" y2="142.24" width="0.1524" layer="91"/>
+<pinref part="U2" gate="G$1" pin="-VIN"/>
+<wire x1="175.26" y1="142.24" x2="180.34" y2="142.24" width="0.1524" layer="91"/>
 <pinref part="C1" gate="G$1" pin="2"/>
-<pinref part="U1" gate="G$1" pin="CAP-"/>
-</segment>
-</net>
-<net name="N$4" class="0">
-<segment>
-<wire x1="180.34" y1="157.48" x2="162.56" y2="157.48" width="0.1524" layer="91"/>
-<pinref part="C1" gate="G$1" pin="1"/>
-<wire x1="162.56" y1="154.94" x2="162.56" y2="157.48" width="0.1524" layer="91"/>
-<pinref part="U1" gate="G$1" pin="CAP+"/>
-</segment>
-</net>
+<wire x1="180.34" y1="142.24" x2="185.42" y2="142.24" width="0.1524" layer="91"/>
+<wire x1="180.34" y1="144.78" x2="180.34" y2="142.24" width="0.1524" layer="91"/>
+<junction x="180.34" y="142.24"/>
+</segment>
+</net>

Commit message: Added power jack.
Parts:
- removed JP2: USB-B, SparkFun-Connectors:USBPTH
- removed U2: DC_ISOLATOR-RKZ0505D, eagle-lib:DC_ISOLATOR-RKZ0505D
- added J4: POWER_JACKPTH, SparkFun-Connectors:POWER_JACKPTH
- added J5: USB-B, SparkFun-Connectors:USBPTH
- added U1: DC_ISOLATOR-RKZ0505D, eagle-lib:DC_ISOLATOR-RKZ0505D
- renumbered JP1 to J6
Connections:
- removed net N$4: C1.2, JP2.GND, U2.-VIN
- new net DGND: C1.2, J4.GND, J5.GND, U1.-VIN
- net +VE: now also U1.+VOUT; no longer U2.+VOUT
- net -VE: now also U1.-VOUT; no longer U2.-VOUT
- net GND: now also U1.COM; no longer U2.COM
- net N$2: now also J4.PWR, J5.VBUS, U1.+VIN; no longer JP2.VBUS, U2.+VIN
Other:
- moved on the sheet: C1, C2, C3
Changed lines of the file:
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@@
 <part name="GND13" library="SparkFun-Aesthetics" deviceset="GND" device=""/>
 <part name="J3" library="eagle-lib" deviceset="M03" device="_0.156IN-RA"/>
-<part name="JP1" library="SparkFun-Connectors" deviceset="M05X2" device="RAF"/>
+<part name="J6" library="SparkFun-Connectors" deviceset="M05X2" device="RAF"/>
 <part name="FRAME1" library="frames" deviceset="FRAME_A_L" device="" value="FRAME"/>
 <part name="U$1" library="ucdrascal-eagle-lib" deviceset="UCDAVIS-RASCAL_LOGO" device="-2LINE"/>
-<part name="U2" library="eagle-lib" deviceset="DC_ISOLATOR" device="-RKZ0505D"/>
-<part name="JP2" library="SparkFun-Connectors" deviceset="USB" device="PTH" value="USB-B"/>
+<part name="U1" library="eagle-lib" deviceset="DC_ISOLATOR" device="-RKZ0505D"/>
+<part name="J5" library="SparkFun-Connectors" deviceset="USB" device="PTH" value="USB-B"/>
 <part name="C1" library="SparkFun-Capacitors" deviceset="CAP" device="0805" value="0.1uF"/>
 <part name="C2" library="SparkFun-Capacitors" deviceset="CAP" device="0805" value="0.1uF"/>
 <part name="C3" library="SparkFun-Capacitors" deviceset="CAP" device="0805" value="0.1uF"/>
+<part name="J4" library="SparkFun-Connectors" deviceset="POWER_JACK" device="PTH"/>
 </parts>
 <sheets>
@@
 <plain>
 <text x="30.48" y="175.26" size="2.54" layer="97">Amplifier Connectors</text>
-<text x="162.56" y="167.64" size="2.54" layer="97">Power Conversion</text>
+<text x="154.94" y="165.1" size="2.54" layer="97">Power Conversion</text>
 <text x="208.28" y="104.14" size="2.54" layer="97">DAQ Connector</text>
 <text x="154.94" y="101.6" size="2.54" layer="97">Reference Electrode</text>
@@
 <instance part="GND13" gate="1" x="243.84" y="78.74"/>
 <instance part="J3" gate="G$1" x="157.48" y="91.44"/>
-<instance part="JP1" gate="G$1" x="226.06" y="88.9"/>
+<instance part="J6" gate="G$1" x="226.06" y="88.9"/>
 <instance part="FRAME1" gate="G$1" x="0" y="0"/>
 <instance part="FRAME1" gate="G$2" x="172.72" y="0"/>
 <instance part="U$1" gate="G$1" x="180.34" y="40.64"/>
-<instance part="U2" gate="G$1" x="200.66" y="147.32"/>
-<instance part="JP2" gate="G$1" x="167.64" y="149.86" rot="MR0"/>
-<instance part="C1" gate="G$1" x="180.34" y="147.32"/>
-<instance part="C2" gate="G$1" x="218.44" y="149.86"/>
-<instance part="C3" gate="G$1" x="220.98" y="142.24"/>
+<instance part="U1" gate="G$1" x="205.74" y="147.32"/>
+<instance part="J5" gate="G$1" x="160.02" y="129.54" rot="MR0"/>
+<instance part="C1" gate="G$1" x="185.42" y="147.32"/>
+<instance part="C2" gate="G$1" x="223.52" y="149.86"/>
+<instance part="C3" gate="G$1" x="226.06" y="142.24"/>
+<instance part="J4" gate="G$1" x="165.1" y="144.78"/>
 </instances>
 <busses>
@@
 <pinref part="GND13" gate="1" pin="GND"/>
 <wire x1="243.84" y1="81.28" x2="243.84" y2="93.98" width="0.1524" layer="91"/>
-<pinref part="JP1" gate="G$1" pin="2"/>
-<pinref part="JP1" gate="G$1" pin="1"/>
+<pinref part="J6" gate="G$1" pin="2"/>
+<pinref part="J6" gate="G$1" pin="1"/>
 <wire x1="218.44" y1="93.98" x2="215.9" y2="93.98" width="0.1524" layer="91"/>
 <wire x1="215.9" y1="93.98" x2="215.9" y2="101.6" width="0.1524" layer="91"/>
@@
 </segment>
 <segment>
-<pinref part="U2" gate="G$1" pin="COM"/>
-<wire x1="215.9" y1="147.32" x2="218.44" y2="147.32" width="0.1524" layer="91"/>
-<label x="231.14" y="147.32" size="1.778" layer="95"/>
+<pinref part="U1" gate="G$1" pin="COM"/>
+<wire x1="220.98" y1="147.32" x2="223.52" y2="147.32" width="0.1524" layer="91"/>
+<label x="236.22" y="147.32" size="1.778" layer="95"/>
 <pinref part="C2" gate="G$1" pin="2"/>
-<wire x1="218.44" y1="147.32" x2="220.98" y2="147.32" width="0.1524" layer="91"/>
-<junction x="218.44" y="147.32"/>
+<wire x1="223.52" y1="147.32" x2="226.06" y2="147.32" width="0.1524" layer="91"/>
+<junction x="223.52" y="147.32"/>
 <pinref part="C3" gate="G$1" pin="1"/>
-<wire x1="220.98" y1="147.32" x2="233.68" y2="147.32" width="0.1524" layer="91"/>
-<junction x="220.98" y="147.32"/>
+<wire x1="226.06" y1="147.32" x2="238.76" y2="147.32" width="0.1524" layer="91"/>
+<junction x="226.06" y="147.32"/>
 </segment>
 </net>
@@
 <wire x1="218.44" y1="91.44" x2="210.82" y2="91.44" width="0.1524" layer="91"/>
 <label x="210.82" y="91.44" size="1.778" layer="95"/>
-<pinref part="JP1" gate="G$1" pin="3"/>
+<pinref part="J6" gate="G$1" pin="3"/>
 </segment>
 <segment>
@@
 <wire x1="218.44" y1="88.9" x2="210.82" y2="88.9" width="0.1524" layer="91"/>
 <label x="210.82" y="88.9" size="1.778" layer="95"/>
-<pinref part="JP1" gate="G$1" pin="5"/>
+<pinref part="J6" gate="G$1" pin="5"/>
 </segment>
 <segment>
@@
 <wire x1="218.44" y1="86.36" x2="210.82" y2="86.36" width="0.1524" layer="91"/>
 <label x="210.82" y="86.36" size="1.778" layer="95"/>
-<pinref part="JP1" gate="G$1" pin="7"/>
+<pinref part="J6" gate="G$1" pin="7"/>
 </segment>
 <segment>
@@
 <wire x1="218.44" y1="83.82" x2="210.82" y2="83.82" width="0.1524" layer="91"/>
 <label x="210.82" y="83.82" size="1.778" layer="95"/>
-<pinref part="JP1" gate="G$1" pin="9"/>
+<pinref part="J6" gate="G$1" pin="9"/>
 </segment>
 <segment>
@@
 <wire x1="233.68" y1="91.44" x2="241.3" y2="91.44" width="0.1524" layer="91"/>
 <label x="237.49" y="91.44" size="1.778" layer="95"/>
-<pinref part="JP1" gate="G$1" pin="4"/>
+<pinref part="J6" gate="G$1" pin="4"/>
 </segment>
 <segment>
@@
 <wire x1="233.68" y1="88.9" x2="241.3" y2="88.9" width="0.1524" layer="91"/>
 <label x="237.49" y="88.9" size="1.778" layer="95"/>
-<pinref part="JP1" gate="G$1" pin="6"/>
+<pinref part="J6" gate="G$1" pin="6"/>
 </segment>
 <segment>
@@
 <wire x1="233.68" y1="86.36" x2="241.3" y2="86.36" width="0.1524" layer="91"/>
 <label x="237.49" y="86.36" size="1.778" layer="95"/>
-<pinref part="JP1" gate="G$1" pin="8"/>
+<pinref part="J6" gate="G$1" pin="8"/>
 </segment>
 <segment>
@@
 <wire x1="233.68" y1="83.82" x2="241.3" y2="83.82" width="0.1524" layer="91"/>
 <label x="237.49" y="83.82" size="1.778" layer="95"/>
-<pinref part="JP1" gate="G$1" pin="10"/>
+<pinref part="J6" gate="G$1" pin="10"/>
 </segment>
 <segment>
@@
 </segment>
 <segment>
-<pinref part="U2" gate="G$1" pin="+VOUT"/>
-<wire x1="215.9" y1="154.94" x2="218.44" y2="154.94" width="0.1524" layer="91"/>
-<label x="231.14" y="154.94" size="1.778" layer="95"/>
+<pinref part="U1" gate="G$1" pin="+VOUT"/>
+<wire x1="220.98" y1="154.94" x2="223.52" y2="154.94" width="0.1524" layer="91"/>
+<label x="236.22" y="154.94" size="1.778" layer="95"/>
 <pinref part="C2" gate="G$1" pin="1"/>
-<wire x1="218.44" y1="154.94" x2="233.68" y2="154.94" width="0.1524" layer="91"/>
-<junction x="218.44" y="154.94"/>
+<wire x1="223.52" y1="154.94" x2="238.76" y2="154.94" width="0.1524" layer="91"/>
+<junction x="223.52" y="154.94"/>
 </segment>
 </net>
@@
 </segment>
 <segment>
-<pinref part="U2" gate="G$1" pin="-VOUT"/>
-<wire x1="215.9" y1="139.7" x2="220.98" y2="139.7" width="0.1524" layer="91"/>
-<label x="231.14" y="139.7" size="1.778" layer="95"/>
+<pinref part="U1" gate="G$1" pin="-VOUT"/>
+<wire x1="220.98" y1="139.7" x2="226.06" y2="139.7" width="0.1524" layer="91"/>
+<label x="236.22" y="139.7" size="1.778" layer="95"/>
 <pinref part="C3" gate="G$1" pin="2"/>
-<wire x1="220.98" y1="139.7" x2="233.68" y2="139.7" width="0.1524" layer="91"/>
-<junction x="220.98" y="139.7"/>
+<wire x1="226.06" y1="139.7" x2="238.76" y2="139.7" width="0.1524" layer="91"/>
+<junction x="226.06" y="139.7"/>
+</segment>
+</net>
+<net name="DGND" class="0">
+<segment>
+<pinref part="U1" gate="G$1" pin="-VIN"/>
+<wire x1="185.42" y1="142.24" x2="190.5" y2="142.24" width="0.1524" layer="91"/>
+<pinref part="C1" gate="G$1" pin="2"/>
+<wire x1="185.42" y1="144.78" x2="185.42" y2="142.24" width="0.1524" layer="91"/>
+<pinref part="J4" gate="G$1" pin="GND"/>
+<wire x1="167.64" y1="147.32" x2="170.18" y2="147.32" width="0.1524" layer="91"/>
+<wire x1="170.18" y1="147.32" x2="170.18" y2="142.24" width="0.1524" layer="91"/>
+<wire x1="170.18" y1="142.24" x2="185.42" y2="142.24" width="0.1524" layer="91"/>
+<junction x="185.42" y="142.24"/>
+<pinref part="J5" gate="G$1" pin="GND"/>
+<wire x1="162.56" y1="129.54" x2="185.42" y2="129.54" width="0.1524" layer="91"/>
+<wire x1="185.42" y1="129.54" x2="185.42" y2="142.24" width="0.1524" layer="91"/>
 </segment>
 </net>
 <net name="N$2" class="0">
 <segment>
-<pinref part="JP2" gate="G$1" pin="VBUS"/>
+<pinref part="U1" gate="G$1" pin="+VIN"/>
 <pinref part="C1" gate="G$1" pin="1"/>
-<wire x1="170.18" y1="152.4" x2="180.34" y2="152.4" width="0.1524" layer="91"/>
-<pinref part="U2" gate="G$1" pin="+VIN"/>
-<wire x1="180.34" y1="152.4" x2="185.42" y2="152.4" width="0.1524" layer="91"/>
-<junction x="180.34" y="152.4"/>
-</segment>
-</net>
-<net name="N$4" class="0">
-<segment>
-<pinref part="JP2" gate="G$1" pin="GND"/>
-<wire x1="170.18" y1="149.86" x2="175.26" y2="149.86" width="0.1524" layer="91"/>
-<wire x1="175.26" y1="149.86" x2="175.26" y2="142.24" width="0.1524" layer="91"/>
-<pinref part="U2" gate="G$1" pin="-VIN"/>
-<wire x1="175.26" y1="142.24" x2="180.34" y2="142.24" width="0.1524" layer="91"/>
-<pinref part="C1" gate="G$1" pin="2"/>
-<wire x1="180.34" y1="142.24" x2="185.42" y2="142.24" width="0.1524" layer="91"/>
-<wire x1="180.34" y1="144.78" x2="180.34" y2="142.24" width="0.1524" layer="91"/>
-<junction x="180.34" y="142.24"/>
-</segment>
-</net>
+<wire x1="190.5" y1="152.4" x2="185.42" y2="152.4" width="0.1524" layer="91"/>
+<pinref part="J4" gate="G$1" pin="PWR"/>
+<junction x="185.42" y="152.4"/>
+<wire x1="167.64" y1="152.4" x2="175.26" y2="152.4" width="0.1524" layer="91"/>
+<pinref part="J5" gate="G$1" pin="VBUS"/>
+<wire x1="175.26" y1="152.4" x2="185.42" y2="152.4" width="0.1524" layer="91"/>
+<wire x1="162.56" y1="132.08" x2="175.26" y2="132.08" width="0.1524" layer="91"/>
+<wire x1="175.26" y1="132.08" x2="175.26" y2="152.4" width="0.1524" layer="91"/>
+<junction x="175.26" y="152.4"/>
+</segment>
+</net>
