File: emg-bridge.sch (EAGLE design)
At the start: 29 parts, among them J1 RJ25_4X1, J2 RJ25_4X1, J3 M03_0.156IN-RA, J4 POWER_JACKPTH, J5 USB-B, J6 M05X2RAF, U1 DC_ISOLATOR-RKZ0505D

Commit message: Minor changes. Revision 1 should really be ready this time.
Parts:
- R17: value (none) -> 1k
Changed lines of the file:
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@@
 <part name="J4" library="SparkFun-Connectors" deviceset="POWER_JACK" device="PTH"/>
 <part name="D1" library="eagle-lib" deviceset="LED" device="_LA93B"/>
-<part name="R17" library="SparkFun-Passives" deviceset="RESISTOR" device="0805-RES"/>
+<part name="R17" library="SparkFun-Passives" deviceset="RESISTOR" device="0805-RES" value="1k"/>
 </parts>
 <sheets>
